File: 6s1pchargeconnector.sch (KiCad schematic (older format))
At the start: 8 parts, among them P1 CONN_01X07, P2 CONN_01X02, P3 CONN_01X02, P4 CONN_01X02, P5 CONN_01X02, P6 CONN_01X02, P7 CONN_01X02, P8 CONN_01X02

Commit message: Added the other two connectors, pcb, gerbers, and bom.
Parts:
- P1: value CONN_01X07 -> CHARGE; footprint Pin_Headers:Pin_Header_Straight_1x07 -> Connectors LEMO:ECG.0B.307; Distributor (none) -> DigiKey; Part Num (none) -> 1124-1321-ND; Price (none) -> 34.73
- P2: value CONN_01X02 -> OUT; Distributor (none) -> SparkFun; Part Num (none) -> PRT-10571; Price (none) -> 0.75
- P3: value CONN_01X02 -> BATT 6; Distributor (none) -> SparkFun; Part Num (none) -> PRT-08612; Price (none) -> 0.95
- P4: value CONN_01X02 -> BATT 5; Distributor (none) -> SparkFun; Part Num (none) -> PRT-08612; Price (none) -> 0.95
- P5: value CONN_01X02 -> BATT 4; Distributor (none) -> SparkFun; Part Num (none) -> PRT-08612; Price (none) -> 0.95
- P6: value CONN_01X02 -> BATT 3; Distributor (none) -> SparkFun; Part Num (none) -> PRT-08612; Price (none) -> 0.95
- P7: value CONN_01X02 -> BATT 2; Distributor (none) -> SparkFun; Part Num (none) -> PRT-08612; Price (none) -> 0.95
- P8: value CONN_01X02 -> BATT 1; Distributor (none) -> SparkFun; Part Num (none) -> PRT-08612; Price (none) -> 0.95
Other:
- note removed: "Possible Connectors:\n7 Pin DIN: CP-3170-ND\n7 Pin Circular: 1124-1321-ND\n"
Changed lines of the file:
@@
 U 1 1 5620653B
 P 5650 4950
-F 0 "P8" H 5650 5100 50  0000 C CNN
-F 1 "CONN_01X02" V 5750 4950 50  0000 C CNN
+F 0 "P8" H 5650 5200 50  0000 C CNN
+F 1 "BATT 1" V 5850 4950 50  0000 C CNN
 F 2 "JST Connectors:JST-PH-2" H 5650 4950 60  0001 C CNN
 F 3 "" H 5650 4950 60  0000 C CNN
+F 4 "SparkFun" H 5650 4950 60  0001 C CNN "Distributor"
+F 5 "PRT-08612" H 5650 4950 60  0001 C CNN "Part Num"
+F 6 "0.95" H 5650 4950 60  0001 C CNN "Price"
 	1    5650 4950
 	1    0    0    -1
@@
 U 1 1 562065CC
 P 5650 4350
-F 0 "P7" H 5650 4500 50  0000 C CNN
-F 1 "CONN_01X02" V 5750 4350 50  0000 C CNN
+F 0 "P7" H 5650 4600 50  0000 C CNN
+F 1 "BATT 2" V 5850 4350 50  0000 C CNN
 F 2 "JST Connectors:JST-PH-2" H 5650 4350 60  0001 C CNN
 F 3 "" H 5650 4350 60  0000 C CNN
+F 4 "SparkFun" H 5650 4350 60  0001 C CNN "Distributor"
+F 5 "PRT-08612" H 5650 4350 60  0001 C CNN "Part Num"
+F 6 "0.95" H 5650 4350 60  0001 C CNN "Price"
 	1    5650 4350
 	1    0    0    -1
@@
 U 1 1 562066AF
 P 5650 3750
-F 0 "P6" H 5650 3900 50  0000 C CNN
-F 1 "CONN_01X02" V 5750 3750 50  0000 C CNN
+F 0 "P6" H 5650 4000 50  0000 C CNN
+F 1 "BATT 3" V 5850 3750 50  0000 C CNN
 F 2 "JST Connectors:JST-PH-2" H 5650 3750 60  0001 C CNN
 F 3 "" H 5650 3750 60  0000 C CNN
+F 4 "SparkFun" H 5650 3750 60  0001 C CNN "Distributor"
+F 5 "PRT-08612" H 5650 3750 60  0001 C CNN "Part Num"
+F 6 "0.95" H 5650 3750 60  0001 C CNN "Price"
 	1    5650 3750
 	1    0    0    -1
@@
 U 1 1 56206742
 P 5650 3150
-F 0 "P5" H 5650 3300 50  0000 C CNN
-F 1 "CONN_01X02" V 5750 3150 50  0000 C CNN
+F 0 "P5" H 5650 3400 50  0000 C CNN
+F 1 "BATT 4" V 5850 3150 50  0000 C CNN
 F 2 "JST Connectors:JST-PH-2" H 5650 3150 60  0001 C CNN
 F 3 "" H 5650 3150 60  0000 C CNN
+F 4 "SparkFun" H 5650 3150 60  0001 C CNN "Distributor"
+F 5 "PRT-08612" H 5650 3150 60  0001 C CNN "Part Num"
+F 6 "0.95" H 5650 3150 60  0001 C CNN "Price"
 	1    5650 3150
 	1    0    0    -1
@@
 U 1 1 56206774
 P 5650 2550
-F 0 "P4" H 5650 2700 50  0000 C CNN
-F 1 "CONN_01X02" V 5750 2550 50  0000 C CNN
+F 0 "P4" H 5650 2800 50  0000 C CNN
+F 1 "BATT 5" V 5850 2550 50  0000 C CNN
 F 2 "JST Connectors:JST-PH-2" H 5650 2550 60  0001 C CNN
 F 3 "" H 5650 2550 60  0000 C CNN
+F 4 "SparkFun" H 5650 2550 60  0001 C CNN "Distributor"
+F 5 "PRT-08612" H 5650 2550 60  0001 C CNN "Part Num"
+F 6 "0.95" H 5650 2550 60  0001 C CNN "Price"
 	1    5650 2550
 	1    0    0    -1
@@
 U 1 1 562067BB
 P 5650 1950
-F 0 "P3" H 5650 2100 50  0000 C CNN
-F 1 "CONN_01X02" V 5750 1950 50  0000 C CNN
+F 0 "P3" H 5650 2200 50  0000 C CNN
+F 1 "BATT 6" V 5850 1950 50  0000 C CNN
 F 2 "JST Connectors:JST-PH-2" H 5650 1950 60  0001 C CNN
 F 3 "" H 5650 1950 60  0000 C CNN
+F 4 "SparkFun" H 5650 1950 60  0001 C CNN "Distributor"
+F 5 "PRT-08612" H 5650 1950 60  0001 C CNN "Part Num"
+F 6 "0.95" H 5650 1950 60  0001 C CNN "Price"
 	1    5650 1950
 	1    0    0    -1
@@
 P 3500 4350
 F 0 "P2" H 3500 4500 50  0000 C CNN
-F 1 "CONN_01X02" V 3600 4350 50  0000 C CNN
+F 1 "OUT" V 3600 4350 50  0000 C CNN
 F 2 "Pin_Headers:Pin_Header_Straight_1x02" H 3500 4350 60  0001 C CNN
 F 3 "" H 3500 4350 60  0000 C CNN
+F 4 "SparkFun" H 3500 4350 60  0001 C CNN "Distributor"
+F 5 "PRT-10571" H 3500 4350 60  0001 C CNN "Part Num"
+F 6 "0.75" H 3500 4350 60  0001 C CNN "Price"
 	1    3500 4350
 	-1   0    0    1
 $EndComp
-Text Notes 7000 6850 0    60   ~ 0
-Possible Connectors:\n7 Pin DIN: CP-3170-ND\n7 Pin Circular: 1124-1321-ND\n
 $Comp
 L CONN_01X07 P1
@@
 P 3500 3400
 F 0 "P1" H 3500 3800 50  0000 C CNN
-F 1 "CONN_01X07" V 3600 3400 50  0000 C CNN
-F 2 "Pin_Headers:Pin_Header_Straight_1x07" H 3500 3400 60  0001 C CNN
+F 1 "CHARGE" V 3600 3400 50  0000 C CNN
+F 2 "Connectors LEMO:ECG.0B.307" H 3500 3400 60  0001 C CNN
 F 3 "" H 3500 3400 60  0000 C CNN
+F 4 "DigiKey" H 3500 3400 60  0001 C CNN "Distributor"
+F 5 "1124-1321-ND" H 3500 3400 60  0001 C CNN "Part Num"
+F 6 "34.73" H 3500 3400 60  0001 C CNN "Price"
 	1    3500 3400
 	-1   0    0    1
